File: mad/mad.sch (KiCad schematic (older format))
At the start: 24 parts, among them X1 Вилка_PLS6, X2 Вилка_PLS6, X3 Вилка_PLS6, X4 Вилка_PLS8

Commit message: незначительные изменения
Connections:
- net labels added: ADC6, ADC7, PC0, PC1, PC2, PC3, PC4, PC5
- wire segments 116 -> 117
Changed lines of the file:
@@
 	4000 2400 2300 2400
-Wire Wire Line
-	2300 2500 4000 2500
 Wire Wire Line
 	2950 2900 2950 2700
@@
 Wire Wire Line
 	4000 2600 3350 2600
-Text Label 2950 2600 0    50   ~ 0
+Text Label 2950 2500 0    50   ~ 0
 VCC_IN
 Wire Wire Line
@@
 Wire Wire Line
 	1600 2500 2300 2500
-Connection ~ 2300 2500
 Wire Wire Line
 	1600 2600 2300 2600
@@
 Wire Wire Line
 	9050 4000 8350 4000
+Text Label 8000 2500 0    50   ~ 0
+ADC6
+Text Label 8000 3000 0    50   ~ 0
+PC2
+Text Label 8000 2900 0    50   ~ 0
+PC1
+Text Label 8000 2800 0    50   ~ 0
+PC0
+Text Label 8000 2700 0    50   ~ 0
+ADC7
+Text Label 8000 3300 0    50   ~ 0
+PC3
+Text Label 8000 3400 0    50   ~ 0
+PC4
+Text Label 8000 3500 0    50   ~ 0
+PC5
+Wire Wire Line
+	3350 2500 4000 2500
+Wire Wire Line
+	2300 2500 2950 2500
+Connection ~ 2300 2500
+Text Label 2950 2600 0    50   ~ 0
+GND
 $EndSCHEMATC
